File: KiCad Schematics/SleepBud/SleepBud.kicad_pcb (KiCad board)
At the start: 2 copper layers, 0 parts

Commit message: Finish Most Footprint, Started Layout
Parts:
- added BT1: Battery_Cell_3V, Battery:BatteryHolder_Keystone_1057_1x2032, F.Cu at (208.0, 72.0)
- added BZ1: PS1240P02BT, digikey-footprints:Piezo_Transducer_THT_PS1240P02BT, F.Cu at (207.0, 96.5)
- added C1: 10uF, Capacitor_SMD:C_0805_2012Metric, F.Cu at (152.6, 79.5)
- added C10: 0.1uF, Capacitor_SMD:C_0603_1608Metric, F.Cu at (172.7, 88.5)
- added C11: 0.1uF, Capacitor_SMD:C_0603_1608Metric, F.Cu at (172.7, 91.0)
- added C12: 0.1uF, Capacitor_SMD:C_0603_1608Metric, F.Cu at (172.7, 93.5)
- added C13: 0.1uF, Capacitor_SMD:C_0603_1608Metric, F.Cu at (172.7, 96.0)
- added C14: 0.1uF, Capacitor_SMD:C_0603_1608Metric, F.Cu at (172.7, 98.5)
- added C2: 22uF, Capacitor_SMD:C_0805_2012Metric, F.Cu at (152.6, 82.5)
- added C3: 10uF, Capacitor_SMD:C_0805_2012Metric, F.Cu at (152.6, 85.5)
- added C4: 22uF, Capacitor_SMD:C_0805_2012Metric, F.Cu at (152.6, 88.5)
- added C5: 1uF, Capacitor_SMD:C_0603_1608Metric, F.Cu at (172.7, 78.4)
- added C6: 22uF, Capacitor_SMD:C_0805_2012Metric, F.Cu at (152.6, 91.5)
- added C7: 0.1uF, Capacitor_SMD:C_0603_1608Metric, F.Cu at (172.7, 80.9)
- added C8: 22pF, Capacitor_SMD:C_0603_1608Metric, F.Cu at (172.7, 83.4)
- added C9: 22pF, Capacitor_SMD:C_0603_1608Metric, F.Cu at (172.7, 86.0)
- added CR1: MBR120LSFT3G, footprints:SDO_SOD-123FL498_OSI, F.Cu at (109.0, 66.0)
- added D10: WS2812B, LED_SMD:LED_WS2812B_PLCC4_5.0x5.0mm_P3.2mm, B.Cu at (126.3, 81.0)
- added D11: WS2812B, LED_SMD:LED_WS2812B_PLCC4_5.0x5.0mm_P3.2mm, B.Cu at (126.1, 86.5)
- added D12: WS2812B, LED_SMD:LED_WS2812B_PLCC4_5.0x5.0mm_P3.2mm, B.Cu at (103.5, 67.9)
- added D13: WS2812B, LED_SMD:LED_WS2812B_PLCC4_5.0x5.0mm_P3.2mm, B.Cu at (103.5, 74.5)
- added D14: WS2812B, LED_SMD:LED_WS2812B_PLCC4_5.0x5.0mm_P3.2mm, B.Cu at (103.5, 81.1)
- added D15: WS2812B, LED_SMD:LED_WS2812B_PLCC4_5.0x5.0mm_P3.2mm, B.Cu at (103.5, 87.7)
- added D16: WS2812B, LED_SMD:LED_WS2812B_PLCC4_5.0x5.0mm_P3.2mm, B.Cu at (103.5, 94.3)
- added D17: WS2812B, LED_SMD:LED_WS2812B_PLCC4_5.0x5.0mm_P3.2mm, B.Cu at (184.6, 61.5)
- added D18: WS2812B, LED_SMD:LED_WS2812B_PLCC4_5.0x5.0mm_P3.2mm, B.Cu at (184.6, 68.1)
- added D19: WS2812B, LED_SMD:LED_WS2812B_PLCC4_5.0x5.0mm_P3.2mm, B.Cu at (184.6, 74.7)
- added D2: WS2812B, LED_SMD:LED_WS2812B_PLCC4_5.0x5.0mm_P3.2mm, B.Cu at (161.7, 60.6)
- added D20: WS2812B, LED_SMD:LED_WS2812B_PLCC4_5.0x5.0mm_P3.2mm, B.Cu at (184.6, 81.3)
- added D21: WS2812B, LED_SMD:LED_WS2812B_PLCC4_5.0x5.0mm_P3.2mm, B.Cu at (184.4, 87.8)
- added D22: WS2812B, LED_SMD:LED_WS2812B_PLCC4_5.0x5.0mm_P3.2mm, B.Cu at (145.2, 76.7)
- added D23: WS2812B, LED_SMD:LED_WS2812B_PLCC4_5.0x5.0mm_P3.2mm, B.Cu at (145.2, 83.3)
- added D24: WS2812B, LED_SMD:LED_WS2812B_PLCC4_5.0x5.0mm_P3.2mm, B.Cu at (184.6, 94.2)
- added D25: WS2812B, LED_SMD:LED_WS2812B_PLCC4_5.0x5.0mm_P3.2mm, B.Cu at (184.6, 100.8)
- added D26: WS2812B, LED_SMD:LED_WS2812B_PLCC4_5.0x5.0mm_P3.2mm, B.Cu at (161.4, 94.3)
- added D27: WS2812B, LED_SMD:LED_WS2812B_PLCC4_5.0x5.0mm_P3.2mm, B.Cu at (161.4, 101.0)
- added D28: WS2812B, LED_SMD:LED_WS2812B_PLCC4_5.0x5.0mm_P3.2mm, B.Cu at (126.0, 93.2)
- added D29: WS2812B, LED_SMD:LED_WS2812B_PLCC4_5.0x5.0mm_P3.2mm, B.Cu at (126.0, 99.8)
- added D3: WS2812B, LED_SMD:LED_WS2812B_PLCC4_5.0x5.0mm_P3.2mm, B.Cu at (161.7, 67.3)
- added D30: WS2812B, LED_SMD:LED_WS2812B_PLCC4_5.0x5.0mm_P3.2mm, B.Cu at (103.5, 100.8)
- added D31: WS2812B, LED_SMD:LED_WS2812B_PLCC4_5.0x5.0mm_P3.2mm, B.Cu at (103.5, 61.4)
- added D4: WS2812B, LED_SMD:LED_WS2812B_PLCC4_5.0x5.0mm_P3.2mm, B.Cu at (161.7, 73.9)
- added D5: WS2812B, LED_SMD:LED_WS2812B_PLCC4_5.0x5.0mm_P3.2mm, B.Cu at (161.7, 80.5)
- added D6: WS2812B, LED_SMD:LED_WS2812B_PLCC4_5.0x5.0mm_P3.2mm, B.Cu at (161.7, 87.1)
- added D7: WS2812B, LED_SMD:LED_WS2812B_PLCC4_5.0x5.0mm_P3.2mm, B.Cu at (126.3, 61.1)
- added D8: WS2812B, LED_SMD:LED_WS2812B_PLCC4_5.0x5.0mm_P3.2mm, B.Cu at (126.3, 67.7)
- added D9: WS2812B, LED_SMD:LED_WS2812B_PLCC4_5.0x5.0mm_P3.2mm, B.Cu at (126.3, 74.3)
- added J1: USB_B_Micro, Connector_USB:USB_Micro-B_Molex-105017-0001, F.Cu at (112.4, 56.8)
- added J2: 12V Barrel Jack, Connector_BarrelJack:BarrelJack_Wuerth_694108106102_2.5x5.5mm, F.Cu at (96.5, 59.9)
- added JP1: UART, Connector_PinHeader_1.00mm:PinHeader_2x02_P1.00mm_Vertical_SMD, F.Cu at (159.5, 57.4)
- added JP2: JTAG, Connector_PinHeader_1.00mm:PinHeader_2x02_P1.00mm_Vertical_SMD, F.Cu at (159.5, 61.5)
- added JP3: Boot Option, Connector_PinHeader_1.00mm:PinHeader_2x01_P1.00mm_Vertical_SMD, F.Cu at (160.8, 72.5)
- added Q1: AO3400A, Package_TO_SOT_SMD:SOT-23, F.Cu at (194.6, 100.0)
- added Q2: FQP27P06, Package_TO_SOT_THT:TO-220-3_Vertical, F.Cu at (81.9, 79.5)
- added R1: 10k, Resistor_SMD:R_1206_3216Metric, F.Cu at (130.8, 87.3)
- added R10: 470, Resistor_SMD:R_1206_3216Metric, F.Cu at (136.4, 93.9)
- added R11: 470, Resistor_SMD:R_1206_3216Metric, F.Cu at (136.4, 97.2)
- added R12: 470, Resistor_SMD:R_1206_3216Metric, F.Cu at (136.4, 100.5)
- added R13: 470, Resistor_SMD:R_1206_3216Metric, F.Cu at (136.4, 103.8)
- added R14: 3.3k, Resistor_SMD:R_0805_2012Metric, F.Cu at (148.1, 99.5)
- added R15: 3.3k, Resistor_SMD:R_0805_2012Metric, F.Cu at (148.1, 102.5)
- added R16: 10k, Resistor_SMD:R_1206_3216Metric, F.Cu at (142.0, 87.3)
- added R17: 10k, Resistor_SMD:R_1206_3216Metric, F.Cu at (142.0, 90.6)
- added R18: 10k, Resistor_SMD:R_1206_3216Metric, F.Cu at (142.0, 93.9)
- added R19: 10k, Resistor_SMD:R_1206_3216Metric, F.Cu at (142.0, 97.2)
- added R2: 470, Resistor_SMD:R_1206_3216Metric, F.Cu at (130.8, 90.6)
- added R20: 10k, Resistor_SMD:R_1206_3216Metric, F.Cu at (142.0, 100.5)
- added R3: 0, Resistor_SMD:R_1206_3216Metric, F.Cu at (130.8, 93.9)
- added R4: 4.7k, Resistor_SMD:R_0201_0603Metric, F.Cu at (165.7, 85.5)
- added R5: 10k, Resistor_SMD:R_1206_3216Metric, F.Cu at (130.8, 97.2)
- added R6: 0, Resistor_SMD:R_1206_3216Metric, F.Cu at (130.8, 100.5)
- added R7: 0, Resistor_SMD:R_1206_3216Metric, F.Cu at (130.8, 103.8)
- added R8: 10kOhm, Resistor_SMD:R_1206_3216Metric, F.Cu at (136.4, 87.3)
- added R9: 470, Resistor_SMD:R_1206_3216Metric, F.Cu at (136.4, 90.6)
- added SW1: Mode Button, Button_Switch_SMD:SW_SPST_B3S-1000, F.Cu at (72.0, 58.9)
- added SW2: Up Button, Button_Switch_SMD:SW_SPST_B3S-1000, F.Cu at (72.0, 67.3)
- added SW3: Down Button, Button_Switch_SMD:SW_SPST_B3S-1000, F.Cu at (72.0, 75.8)
- added SW4: EN Button, Button_Switch_SMD:SW_Tactile_SPST_NO_Straight_CK_PTS636Sx25SMTRLFS, F.Cu at (121.1, 65.5)
- added SW5: Switch Button, Button_Switch_SMD:SW_SPST_B3S-1000, F.Cu at (72.0, 84.2)
- added SW6: Reset Button, Button_Switch_SMD:SW_Tactile_SPST_NO_Straight_CK_PTS636Sx25SMTRLFS, F.Cu at (169.1, 66.0)
- added U1: ESP32-S3-WROOM-1, RF_Module:ESP32-S3-WROOM-1, F.Cu at (143.5, 61.0)
- added U2: DS3231SN_, DS3231SN_:SOIC127P1032X265-16N, F.Cu at (181.2, 66.6)
- added U3: PIR, Connector_PinHeader_1.00mm:PinHeader_1x03_P1.00mm_Vertical_SMD_Pin1Left, F.Cu at (129.6, 66.0)
- added U4: AMS1117-3.3, Package_TO_SOT_SMD:SOT-223-3_TabPin2, F.Cu at (96.8, 74.7)
- added U5: AMS1117-5.0, Package_TO_SOT_SMD:SOT-223-3_TabPin2, F.Cu at (96.8, 83.0)
- added U6: TXS0108EPW, Package_SO:TSSOP-20_4.4x6.5mm_P0.65mm, F.Cu at (119.5, 84.5)
- added U7: Lamp SMD, Connector_PinHeader_1.00mm:PinHeader_1x03_P1.00mm_Vertical_SMD_Pin1Right, F.Cu at (108.1, 97.0)
Other:
- board outline added: 155 x 55 mm
- board text added: "11/6/2024"
- board text added: "Team 3 SleepBud Version 1"
