File: KiCad Schematics/SleepBud/SleepBud.kicad_sch (KiCad schematic)
At the start: 6 parts, among them U1 ESP32-S3-WROOM-1, U2 DS3231SN_, U3 AM312, U4 AMS1117-3.3, U5 AMS1117-5.0

Commit message: Version 10/25
Added connections
Parts:
- removed BZ1: Buzzer, symbol Device:Buzzer
- added C1, C3: 10uF, symbol Device:C
- added C2, C4, C6: 22uF, symbol Device:C
- added C5: 1uF, symbol Device:C
- added C7: 0.1uF, symbol Device:C
- added C8, C9: TBD, symbol Device:C
- added D1, D10, D11, D12, D13, D14, D15, D16, D17, D18, D19, D2, D20, D21, D22, D23, D24, D25, D26, D27, D28, D29, D3, D30, D31, D32, D33, D34, D35, D36, D37, D38, D39, D4, D40, D41, D42, D43, D44, D45, D46, D47, D48, D49, D5, D50, D6, D7, D8, D9: WS2812B, LED_SMD:LED_WS2812B_PLCC4_5.0x5.0mm_P3.2mm, symbol LED:WS2812B
- added J1: USB_B_Micro, symbol Connector:USB_B_Micro
- added LS1: Speaker, symbol Device:Speaker
- added R1, R2, R3, R4: 470, symbol Device:R
- added R5: 10k, symbol Device:R
- added R6, R7: 0, symbol Device:R
- added SW1, SW2, SW3: SW_Push, symbol Switch:SW_Push
Connections:
- net GND: now reaches U2.13 (GND)
- net GND: now also U1.1 (GND), U1.40 (GND), U1.41 (GND), U3.1 (VCC), U4.1 (GND), U5.1 (GND), C1.2, C2.2, C3.2, C4.2, C5.1, C6.2, C7.2, C8.2, C9.2, D1.3 (VSS), D32.3 (VSS), D33.3 (VSS), D34.3 (VSS), D35.3 (VSS), D36.3 (VSS), D37.3 (VSS), D38.3 (VSS), D39.3 (VSS), D40.3 (VSS), D41.3 (VSS), D42.3 (VSS), D43.3 (VSS), D44.3 (VSS), D45.3 (VSS), D46.3 (VSS), D47.3 (VSS), D48.3 (VSS), D49.3 (VSS), D50.3 (VSS), J1.5 (GND), J1.6 (Shield), LS1.2
- net +5V: now reaches U5.2 (VO)
- net +5V: now also C4.1, D1.1 (VDD), D32.1 (VDD), D33.1 (VDD), D34.1 (VDD), D35.1 (VDD), D36.1 (VDD), D37.1 (VDD), D38.1 (VDD), D39.1 (VDD), D40.1 (VDD), D41.1 (VDD), D42.1 (VDD), D43.1 (VDD), D44.1 (VDD), D45.1 (VDD), D46.1 (VDD), D47.1 (VDD), D48.1 (VDD), D49.1 (VDD), D50.1 (VDD)
- net +12V: now reaches U5.3 (VI)
- net +12V: now also U4.3 (VI), C1.1, C3.1
- net at U1.13 (IO19): now also R6.1
- net at U1.14 (IO20): now also R7.1
- net +3.3V: now reaches U1.2 (3V3)
- net +3.3V: now also U3.3 (GND), U4.2 (VO), C2.1, C6.1, C7.1, R5.1
- net at U1.3 (EN): now also C5.2, R5.2
- new net: D37.2 (DOUT), D38.4 (DIN)
- new net: D36.2 (DOUT), D37.4 (DIN)
- new net: D44.2 (DOUT), D45.4 (DIN)
- new net: D43.2 (DOUT), D44.4 (DIN)
- new net: D1.4 (DIN), R3.2
- new net: D41.4 (DIN), R1.2
- new net: D1.2 (DOUT), D32.4 (DIN)
- new net: D39.2 (DOUT), D40.4 (DIN)
- new net: D38.2 (DOUT), D39.4 (DIN)
- new net: D33.2 (DOUT), D34.4 (DIN)
- new net: D32.2 (DOUT), D33.4 (DIN)
- new net: D47.2 (DOUT), D48.4 (DIN)
- new net: D46.2 (DOUT), D47.4 (DIN)
- new net: C9.1, J1.3 (D+), R7.2
- new net: D42.2 (DOUT), D43.4 (DIN)
- new net: D41.2 (DOUT), D42.4 (DIN)
- new net: D49.2 (DOUT), D50.4 (DIN)
- new net: D48.2 (DOUT), D49.4 (DIN)
- new net: D34.2 (DOUT), D35.4 (DIN)
- new net: D46.4 (DIN), R2.2
- new net: D36.4 (DIN), R4.2
- new net: C8.1, J1.2 (D-), R6.2
- no-connect marks 0 -> 4
Other:
- note added: "4 LED on a Strips w/ 4-7 Strips... Still deciding how many in a strip"
- note added: "7 Segment LED"
- note added: "Barrel Jack Power Supply 12V/5A"
- note added: "Buttons"
- note added: "Goes to LEDs"
- note added: "Goes to the rest of the PCB"
- note added: "LED LAMP"
- note added: "Power Supply"
- note added: "Speaker"
- note added: "USB"
- moved on the sheet: U1, U2, U3, U4, U5

Commit message: new version with updated stuff
Other:
- note added: "SleepBud"
- note added: "TO DO: Connect 7 Segment LED Connect LED Lamp to ESP32 Finish schematic ESP32 Once schematic of ESP32 is done connect actuators and sensors to ESP32"

Commit message: new
Parts:
- added J2: 12V, symbol Connector:Barrel_Jack
Connections:
- net GND: now also J2.2
- net +12V: no longer names the net of C1.1, C3.1, U4.3 (VI), U5.3 (VI)
- net +12V: now also J2.1
Other:
- note added: "Front Side of The PCB (the IC side)"
- note added: "Not Part of PCB (LEDs only) just what it would the parts would be needed for the Lamp"
- note added: "Other Side of the PCB Board"
Changed lines of the file:
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@@
 	)
 	(junction
+		(at 29.21 49.53)
+		(diameter 0)
+		(color 0 0 0 0)
+	)
+	(junction
 		(at 63.5 24.13)
 		(diameter 0)
@@
 	)
 	(junction
-		(at 25.4 54.61)
-		(diameter 0)
-		(color 0 0 0 0)
-	)
-	(junction
 		(at 72.39 196.85)
 		(diameter 0)
@@
 	)
 	(junction
-		(at 102.87 170.18)
+		(at 25.4 43.18)
 		(diameter 0)
 		(color 0 0 0 0)
 	)
 	(junction
-		(at 140.97 29.21)
+		(at 102.87 170.18)
 		(diameter 0)
 		(color 0 0 0 0)
 	)
 	(junction
-		(at 25.4 49.53)
+		(at 140.97 29.21)
 		(diameter 0)
 		(color 0 0 0 0)
@@
 	(wire
 		(pts
-			(xy 25.4 54.61) (xy 25.4 73.66)
-		)
-		(stroke
-			(width 0)
-			(type default)
-		)
-	)
-	(wire
-		(pts
 			(xy 87.63 212.09) (xy 102.87 212.09)
 		)
@@
 	(wire
 		(pts
-			(xy 25.4 49.53) (xy 25.4 54.61)
-		)
-		(stroke
-			(width 0)
-			(type default)
-		)
-	)
-	(wire
-		(pts
 			(xy 181.61 52.07) (xy 190.5 52.07)
 		)
@@
 	(wire
 		(pts
+			(xy 25.4 57.15) (xy 29.21 57.15)
+		)
+		(stroke
+			(width 0)
+			(type default)
+		)
+	)
+	(wire
+		(pts
 			(xy 102.87 175.26) (xy 118.11 175.26)
 		)
@@
 	(wire
 		(pts
+			(xy 25.4 57.15) (xy 25.4 73.66)
+		)
+		(stroke
+			(width 0)
+			(type default)
+		)
+	)
+	(wire
+		(pts
 			(xy 205.74 54.61) (xy 205.74 57.15)
 		)
@@
 	(wire
 		(pts
+			(xy 29.21 43.18) (xy 29.21 49.53)
+		)
+		(stroke
+			(width 0)
+			(type default)
+		)
+	)
+	(wire
+		(pts
 			(xy 118.11 170.18) (xy 133.35 170.18)
 		)
@@
 	(wire
 		(pts
+			(xy 25.4 43.18) (xy 29.21 43.18)
+		)
+		(stroke
+			(width 0)
+			(type default)
+		)
+	)
+	(wire
+		(pts
 			(xy 72.39 212.09) (xy 87.63 212.09)
 		)
@@
 	(wire
 		(pts
+			(xy 29.21 49.53) (xy 29.21 57.15)
+		)
+		(stroke
+			(width 0)
+			(type default)
+		)
+	)
+	(wire
+		(pts
 			(xy 102.87 170.18) (xy 118.11 170.18)
 		)
@@
 	(wire
 		(pts
-			(xy 25.4 24.13) (xy 25.4 49.53)
+			(xy 25.4 24.13) (xy 25.4 43.18)
 		)
 		(stroke
@@
 		)
 	)
+	(text "Front Side of The PCB (the IC side)"
+		(exclude_from_sim no)
+		(at 31.242 104.394 0)
+		(effects
+			(font
+				(size 1.27 1.27)
+				(thickness 0.254)
+				(bold yes)
+			)
+		)
+	)
 	(text "Voltage Regulator\n"
 		(exclude_from_sim no)
@@
 		)
 	)
+	(text "Not Part of PCB (LEDs only) just what it\nwould the parts would be needed for the Lamp\n"
+		(exclude_from_sim no)
+		(at 133.858 255.27 0)
+		(effects
+			(font
+				(size 1.27 1.27)
+				(thickness 0.254)
+				(bold yes)
+			)
+		)
+	)
+	(text "Other Side of the PCB Board\n"
+		(exclude_from_sim no)
+		(at 210.058 232.41 0)
+		(effects
+			(font
+				(size 1.27 1.27)
+				(thickness 0.254)
+				(bold yes)
+			)
+		)
+	)
 	(text "4 LED on a Strips w/\n4-7 Strips... Still deciding how many in a strip\n\n"
 		(exclude_from_sim no)
@@
 		(on_board yes)
 		(dnp no)
-		(fields_autoplaced yes)
 		(property "Reference" "SW3"
 			(at 121.92 77.47 0)
@@
 	(symbol
 		(lib_id "power:PWR_FLAG")
-		(at 25.4 49.53 270)
+		(at 29.21 49.53 270)
 		(unit 1)
 		(exclude_from_sim no)
@@
 		(fields_autoplaced yes)
 		(property "Reference" "#FLG01"
-			(at 27.305 49.53 0)
+			(at 31.115 49.53 0)
 			(effects
 				(font
@@
 		)
 		(property "Value" "PWR_FLAG"
-			(at 29.21 49.5299 90)
+			(at 33.02 49.5299 90)
 			(effects
 				(font
@@
 		)
 		(property "Footprint" ""
-			(at 25.4 49.53 0)
+			(at 29.21 49.53 0)
 			(effects
 				(font
@@
 		)
 		(property "Datasheet" "~"
-			(at 25.4 49.53 0)
+			(at 29.21 49.53 0)
 			(effects
 				(font
@@
 		)
 		(property "Description" "Special symbol for telling ERC where power comes from"
-			(at 25.4 49.53 0)
+			(at 29.21 49.53 0)
 			(effects
 				(font
@@
 	)
 	(symbol
-		(lib_id "power:+12V")
-		(at 25.4 54.61 90)
-		(unit 1)
-		(exclude_from_sim no)
-		(in_bom yes)
-		(on_board yes)
-		(dnp no)
-		(property "Reference" "#PWR01"
-			(at 29.21 54.61 0)
-			(effects
-				(font
-					(size 1.27 1.27)
-				)
-				(hide yes)
-			)
-		)
-		(property "Value" "+12V"
-			(at 21.59 54.6099 90)
-			(effects
-				(font
-					(size 1.27 1.27)
-				)
-				(justify left)
-			)
-		)
-		(property "Footprint" ""
-			(at 25.4 54.61 0)
-			(effects
-				(font
-					(size 1.27 1.27)
-				)
-				(hide yes)
-			)
-		)
-		(property "Datasheet" ""
-			(at 25.4 54.61 0)
-			(effects
-				(font
-					(size 1.27 1.27)
-				)
-				(hide yes)
-			)
-		)
-		(property "Description" "Power symbol creates a global label with name \"+12V\""
-			(at 25.4 54.61 0)
-			(effects
-				(font
-					(size 1.27 1.27)
-				)
-				(hide yes)
-			)
-		)
-		(pin "1"
-		)
-		(instances
-			(project ""
-				(path "/976e55d6-47c8-4a6a-a3ac-d81121411704"
-					(reference "#PWR01")
-					(unit 1)
-				)
-			)
-		)
-	)
-	(symbol
 		(lib_id "AMC312_Mini_PIR:AM312")
 		(at 102.87 71.12 180)
@@
 	)
 	(symbol
+		(lib_id "Connector:Barrel_Jack")
+		(at 17.78 45.72 0)
+		(unit 1)
+		(exclude_from_sim no)
+		(in_bom yes)
+		(on_board yes)
+		(dnp no)
+		(fields_autoplaced yes)
+		(property "Reference" "J2"
+			(at 17.78 36.83 0)
+			(effects
+				(font
+					(size 1.27 1.27)
+				)
+			)
+		)
+		(property "Value" "12V"
+			(at 17.78 39.37 0)
+			(effects
+				(font
+					(size 1.27 1.27)
+				)
+			)
+		)
+		(property "Footprint" ""
+			(at 19.05 46.736 0)
+			(effects
+				(font
+					(size 1.27 1.27)
+				)
+				(hide yes)
+			)
+		)
+		(property "Datasheet" "~"
+			(at 19.05 46.736 0)
+			(effects
+				(font
+					(size 1.27 1.27)
+				)
+				(hide yes)
+			)
+		)
+		(property "Description" "DC Barrel Jack"
+			(at 17.78 45.72 0)
+			(effects
+				(font
+					(size 1.27 1.27)
+				)
+				(hide yes)
+			)
+		)
+		(pin "1"
+		)
+		(pin "2"
+		)
+		(instances
+			(project ""
+				(path "/976e55d6-47c8-4a6a-a3ac-d81121411704"
+					(reference "J2")
+					(unit 1)
+				)
+			)
+		)
+	)
+	(symbol
 		(lib_id "LED:WS2812B")
 		(at 87.63 204.47 0)
@@
 					(unit 1)
 				)
+			)
+		)
+	)
+	(symbol
+		(lib_id "power:GND")
+		(at 25.4 48.26 0)
+		(unit 1)
+		(exclude_from_sim no)
+		(in_bom yes)
+		(on_board yes)
+		(dnp no)
+		(fields_autoplaced yes)
+		(property "Reference" "#PWR01"
+			(at 25.4 54.61 0)
+			(effects
+				(font
+					(size 1.27 1.27)
+				)
+				(hide yes)
+			)
+		)
+		(property "Value" "GND"
+			(at 25.4 53.34 0)
+			(effects
+				(font
+					(size 1.27 1.27)
+				)
+			)
+		)
+		(property "Footprint" ""
+			(at 25.4 48.26 0)
+			(effects
+				(font
+					(size 1.27 1.27)
+				)
+				(hide yes)
+			)
+		)
+		(property "Datasheet" ""
+			(at 25.4 48.26 0)
+			(effects
+				(font
+					(size 1.27 1.27)
+				)
+				(hide yes)
+			)
+		)
+		(property "Description" "Power symbol creates a global label with name \"GND\" , ground"
+			(at 25.4 48.26 0)
+			(effects
+				(font
+					(size 1.27 1.27)
+				)
+				(hide yes)
+			)
+		)
+		(pin "1"
+		)
+		(instances
+			(project ""
+				(path "/976e55d6-47c8-4a6a-a3ac-d81121411704"
+					(reference "#PWR01")
+					(unit 1)
+				)

Commit message: SleepBud Schematic 11/1/2024
Parts:
- added BT1: Battery_Cell_3V, symbol Device:Battery_Cell
- added C10, C11: 0.1uF, symbol Device:C
- added D51, D52, D53, D54, D55, D56, D57, D58, D59, D60, D61, D62, D63, D64, D65, D66, D67, D68, D69, D70, D71, D72, D73, D74, D75, D76, D77, D78: WS2812B, LED_SMD:LED_WS2812B_PLCC4_5.0x5.0mm_P3.2mm, symbol LED:WS2812B
- added R10, R11, R12, R13, R9: 470, symbol Device:R
- added R8: 10kOhm, symbol Device:R
- added U6: TXS0108EPW, Package_SO:TSSOP-20_4.4x6.5mm_P0.65mm, symbol Logic_LevelTranslator:TXS0108EPW
Connections:
- net +3.3V: now also U2.2 (VCC), C10.1, U6.2 (VCCA)
- net +5V: now also D10.1 (VDD), D11.1 (VDD), D12.1 (VDD), D13.1 (VDD), D14.1 (VDD), D15.1 (VDD), D16.1 (VDD), D17.1 (VDD), D18.1 (VDD), D19.1 (VDD), D2.1 (VDD), D20.1 (VDD), D21.1 (VDD), D22.1 (VDD), D23.1 (VDD), D24.1 (VDD), D25.1 (VDD), D26.1 (VDD), D27.1 (VDD), D28.1 (VDD), D29.1 (VDD), D3.1 (VDD), D30.1 (VDD), D31.1 (VDD), D4.1 (VDD), D5.1 (VDD), D6.1 (VDD), D7.1 (VDD), D8.1 (VDD), D9.1 (VDD), C11.1, D51.1 (VDD), D52.1 (VDD), D53.1 (VDD), D54.1 (VDD), D55.1 (VDD), D56.1 (VDD), D57.1 (VDD), D58.1 (VDD), D59.1 (VDD), D60.1 (VDD), D61.1 (VDD), D62.1 (VDD), D63.1 (VDD), D64.1 (VDD), D65.1 (VDD), D66.1 (VDD), D67.1 (VDD), D68.1 (VDD), D69.1 (VDD), D70.1 (VDD), D71.1 (VDD), D72.1 (VDD), D73.1 (VDD), D74.1 (VDD), D75.1 (VDD), D76.1 (VDD), D77.1 (VDD), D78.1 (VDD), U6.19 (VCCB)
- net GND: now also D10.3 (VSS), D11.3 (VSS), D12.3 (VSS), D13.3 (VSS), D14.3 (VSS), D15.3 (VSS), D16.3 (VSS), D17.3 (VSS), D18.3 (VSS), D19.3 (VSS), D2.3 (VSS), D20.3 (VSS), D21.3 (VSS), D22.3 (VSS), D23.3 (VSS), D24.3 (VSS), D25.3 (VSS), D26.3 (VSS), D27.3 (VSS), D28.3 (VSS), D29.3 (VSS), D3.3 (VSS), D30.3 (VSS), D31.3 (VSS), D4.3 (VSS), D5.3 (VSS), D6.3 (VSS), D7.3 (VSS), D8.3 (VSS), D9.3 (VSS), BT1.2 (-), C10.2, C11.2, D51.3 (VSS), D52.3 (VSS), D53.3 (VSS), D54.3 (VSS), D55.3 (VSS), D56.3 (VSS), D57.3 (VSS), D58.3 (VSS), D59.3 (VSS), D60.3 (VSS), D61.3 (VSS), D62.3 (VSS), D63.3 (VSS), D64.3 (VSS), D65.3 (VSS), D66.3 (VSS), D67.3 (VSS), D68.3 (VSS), D69.3 (VSS), D70.3 (VSS), D71.3 (VSS), D72.3 (VSS), D73.3 (VSS), D74.3 (VSS), D75.3 (VSS), D76.3 (VSS), D77.3 (VSS), D78.3 (VSS), R8.2, U6.11 (GND)
- net at D22.2 (DOUT): now also D23.4 (DIN)
- net at D22.4 (DIN): now also R13.2
- net at D7.2 (DOUT): now also D8.4 (DIN)
- net at D7.4 (DIN): now also R10.2
- net at D10.2 (DOUT): now also D11.4 (DIN)
- net at D10.4 (DIN): now also D9.2 (DOUT)
- net at D3.2 (DOUT): now also D4.4 (DIN)
- net at D3.4 (DIN): now also D2.2 (DOUT)
- net at D24.2 (DOUT): now also D25.4 (DIN)
- net at D24.4 (DIN): now also D21.2 (DOUT)
- net at R3.2: now also D43.4 (DIN); no longer D1.4 (DIN)
- net at D41.4 (DIN): now also D40.2 (DOUT); no longer R1.2
- net at D13.2 (DOUT): now also D14.4 (DIN)
- net at D13.4 (DIN): now also D12.2 (DOUT)
- net at D15.2 (DOUT): now also D16.4 (DIN)
- net at D15.4 (DIN): now also D14.2 (DOUT)
- net at D6.4 (DIN): now also D5.2 (DOUT)
- net at D12.4 (DIN): now also R11.2
- net at D8.2 (DOUT): now also D9.4 (DIN)
- net at D21.4 (DIN): now also D20.2 (DOUT)
- net at D29.4 (DIN): now also D28.2 (DOUT)
- net at D42.2 (DOUT): no longer D43.4 (DIN)
- net at D17.2 (DOUT): now also D18.4 (DIN)
- net at D17.4 (DIN): now also R12.2
- net at D26.2 (DOUT): now also D27.4 (DIN)
- net at D20.4 (DIN): now also D19.2 (DOUT)
- net at D19.4 (DIN): now also D18.2 (DOUT)
- net at D30.2 (DOUT): now also D31.4 (DIN)
- net at D45.2 (DOUT): now also D58.4 (DIN)
- net at D5.4 (DIN): now also D4.2 (DOUT)
- net at U2.14 (VBAT): now also BT1.1 (+)
- net at D35.2 (DOUT): now also D36.4 (DIN)
- net at D50.2 (DOUT): now also D51.4 (DIN)
- net at R4.2: now also D67.4 (DIN); no longer D36.4 (DIN)
- net at D2.4 (DIN): now also R9.2
- net VBUS: now reaches J1.1 (VBUS)
- new net: D77.2 (DOUT), D78.4 (DIN)
- new net: D76.2 (DOUT), D77.4 (DIN)
- new net: D64.2 (DOUT), D65.4 (DIN)
- new net: D63.2 (DOUT), D64.4 (DIN)
- new net: R8.1, U6.10 (OE)
- new net: D71.2 (DOUT), D72.4 (DIN)
- new net: D70.2 (DOUT), D71.4 (DIN)
- new net: D55.2 (DOUT), D56.4 (DIN)
- new net: D54.2 (DOUT), D55.4 (DIN)
- new net: D73.2 (DOUT), D74.4 (DIN)
- new net: D72.2 (DOUT), D73.4 (DIN)
- new net: D65.2 (DOUT), D66.4 (DIN)
- new net: D67.2 (DOUT), D68.4 (DIN)
- new net: D60.2 (DOUT), D61.4 (DIN)
- new net: D59.2 (DOUT), D60.4 (DIN)
- new net: D75.2 (DOUT), D76.4 (DIN)
- new net: D62.2 (DOUT), D63.4 (DIN)
- new net: D61.2 (DOUT), D62.4 (DIN)
- new net: D56.2 (DOUT), D57.4 (DIN)
- new net: D68.2 (DOUT), D69.4 (DIN)
- new net: D74.2 (DOUT), D75.4 (DIN)
- new net: D1.4 (DIN), R1.2
- new net: D53.2 (DOUT), D54.4 (DIN)
- new net: D52.2 (DOUT), D53.4 (DIN)
- new net: D51.2 (DOUT), D52.4 (DIN)
- new net: D69.2 (DOUT), D70.4 (DIN)
- new net: D58.2 (DOUT), D59.4 (DIN)
- no-connect marks 4 -> 11
Other:
- note added: "12 LED on a Strips w/ 4-7 Strips... Still deciding how many in a strip"
- note added: "Barrel Jack Power Supply 12V/3A"
- note added: "Team 3"
- note added: "Version 1"
- note removed: "4 LED on a Strips w/ 4-7 Strips... Still deciding how many in a strip"
- note removed: "Barrel Jack Power Supply 12V/5A"
- moved on the sheet: D46, D47, D48, D49, D50, LS1, R2, U2

Commit message: Version 1.1
Parts:
- removed R3, R4: 470, symbol Device:R
- added CR1: MBR120LSFT3G, SDO_SOD-123FL498_OSI, symbol MBR120LSFT3G:MBR120LSFT3G
- added Q1: AO3400A, Package_TO_SOT_SMD:SOT-23, symbol Transistor_FET:AO3400A
- added Q2: FQP27P06, Package_TO_SOT_THT:TO-220-3_Vertical, symbol Transistor_FET:FQP27P06
- added SW4, SW5, SW6: SW_Push, symbol Switch:SW_Push
- R1: value 470 -> 10k
- SW1: value SW_Push -> Mode
- SW2: value SW_Push -> Up Button
- SW3: value SW_Push -> Down Button
Connections:
- net GND: now also R1.2
- net RW1-RW2: now also D1.4 (DIN), D57.2 (DOUT)
- net RW2-RW3: now also D42.2 (DOUT), D43.4 (DIN)
- net RW3-RW4: now also D66.2 (DOUT), D67.4 (DIN)
- net VBUS: now also R1.1, CR1.2, Q2.1 (G)
- net at D30.4 (DIN): now also D16.2 (DOUT)
- net at D26.4 (DIN): now also D6.2 (DOUT)
- net at D11.2 (DOUT): now also D28.4 (DIN)
- net at C3.1, J2.1, U5.3 (VI): now also Q2.2 (D); no longer C1.1, U4.3 (VI)
- net at U6.1 (A1): now also U1.22 (IO14)
- net Digit 4: now reaches U6.14 (B6)
- net Digit 4: now also R11.1
- net Digit 3: now reaches U6.15 (B5)
- net Digit 3: now also R10.1
- net Colon: now reaches U6.16 (B4)
- net Colon: now also R13.1
- net Digit 2: now reaches U6.17 (B3)
- net Digit 2: now also R9.1
- net Digit 1: now reaches U6.18 (B2)
- net Digit 1: now also R12.1
- net LED Lamp: now reaches U6.20 (B1)
- net LED Lamp: now also R2.1
- net at U6.3 (A2): now also U1.21 (IO13)
- net at U6.4 (A3): now also U1.20 (IO12)
- net at U6.5 (A4): now also U1.19 (IO11)
- net at U6.6 (A5): now also U1.18 (IO10)
- net at U6.7 (A6): now also U1.17 (IO9)
- new net: C1.1, CR1.1, Q2.3 (S), U4.3 (VI)
- no-connect marks 11 -> 14
Other:
- note added: "12 LED on a Strips w/ 4 Strips"
- note added: "TO DO: Finish schematic ESP32 Once schematic of ESP32 is done connect actuators and sensors to ESP32"
- note added: "Version 1.2"
- note added: "can change diode if need be"
- note removed: "12 LED on a Strips w/ 4-7 Strips... Still deciding how many in a strip"
- note removed: "TO DO: Connect 7 Segment LED Connect LED Lamp to ESP32 Finish schematic ESP32 Once schematic of ESP32 is done connect actuators and sensors to ESP32"
- note removed: "Version 1"
- moved on the sheet: C1, C10, C2, C3, C4, D26, D27, D28, D29, D30, D31, J2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

Commit message: Finished Wiring Schematic
Wiring is finished, however there are 10 errors left that need to be checked/ fixed
Parts:
- removed LS1: Speaker, symbol Device:Speaker
- added BZ1: PS1240P02BT, digikey-footprints:Piezo_Transducer_THT_PS1240P02BT, symbol dk_Alarms-Buzzers-and-Sirens:PS1240P02BT
- added C12, C13, C14: 0.1uF, symbol Device:C
- added JP1: UART, symbol UART Pads:UART
- added JP2: JTAG, symbol JTAG Pads:JTAG_PAD
- added JP3: Boot Option, symbol Boot Option:Boot_Option
- added R14, R15: 3.3k, symbol Device:R
- added R16, R17, R18, R19, R20: 10k, symbol Device:R
- added R3: 0, symbol Device:R
- added R4: 4.7k, symbol Device:R
- SW4: value SW_Push -> EN Button
- U3: value AM312 -> PIR
Connections:
- net +3.3V: now also U2.15 (SDA), U2.16 (SCL), U3.1 (VCC), C14.1, JP1.1 (VCC), R14.1, R15.1, R17.1, R18.1, R19.1, R20.1, R4.1; no longer U3.3 (GND)
- net GND: now also Q1.2 (S), SW1.1, SW2.1, SW3.1, SW4.1, SW5.1, SW6.1, U3.3 (GND), C12.1, C13.2, C14.2, JP1.4 (GND), JP3.2 (GND); no longer U3.1 (VCC)
- net at R8.1, U6.10 (OE): now also U1.31 (IO38)
- net at Q1.1 (G): now also R16.2
- net at Q1.3 (D): now also BZ1.2
- net at SW1.2: now also U1.4 (IO4), R17.2
- net +12V: now reaches C3.1, J2.1, Q2.2 (D), U5.3 (VI)
- net +12V: now also BZ1.1
- net at SW3.2: now also U1.6 (IO6), R19.2
- net at C5.2, R5.2, U1.3 (EN): now also R3.2
- net at SW5.2: now also U1.7 (IO7), R20.2
- net at BT1.1 (+), U2.14 (VBAT): now also C13.1
- net at U2.3 (SQW/~{INT}): now also U1.30 (IO37), R4.2
- net at U2.4 (~{RST}): now also SW6.2
- net at SW4.2: now also C12.2, R3.1
- net at U1.12 (IO8): now also U3.2 (PIR_Signal)
- net Buzzer: now reaches U1.23 (IO21)
- net Buzzer: now also R16.1
- net at U1.27 (IO0): now also JP3.1 (Input)
- net at U1.28 (IO35): now also R14.2
- net at U1.29 (IO36): now also R15.2
- net at U1.32 (IO39): now also JP2.4 (TCK)
- net at U1.33 (IO40): now also JP2.3 (TDO)
- net at U1.34 (IO41): now also JP2.2 (TDI)
- net at U1.35 (IO42): now also JP2.1 (TMS)
- net at U1.36 (RXD0): now also JP1.3 (RXD0)
- net at U1.37 (TXD0): now also JP1.2 (TXD0)
- net at U1.5 (IO5): now also SW2.2, R18.2
- no-connect marks 14 -> 23
Other:
- note added: "Buzzer"
- note removed: "Speaker"
- note removed: "TO DO: Finish schematic ESP32 Once schematic of ESP32 is done connect actuators and sensors to ESP32"
- moved on the sheet: BT1, C1, C5, C6, C7, Q1, R1, R5, SW1, SW2, SW3, SW4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
