File: KiCad Schematics/SleepBud/SleepBud.kicad_sch (KiCad schematic)
At the start: 163 parts, among them J1 12V Barrel Jack, J2 USB_B_Micro, J3 Button Connector, J4 AM312 Connector, J5 LED Lamp Connector, J6 Connector to Buzzer, Q1 DMG3415U-7, Q2 AO3400A, SW1 EN Button, SW2 Reset Button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

Commit message: chnaged power supply once more
Other:
- note added: "Barrel Jack Power Supply 5V/4A"
- note removed: "Barrel Jack Power Supply 9V/3A"
Changed lines of the file:
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@@
 		)
 	)
-	(text "Barrel Jack Power Supply 9V/3A"
+	(text "Barrel Jack Power Supply 5V/4A"
 		(exclude_from_sim no)
 		(at 63.5 182.626 0)
